Commit message: change box position for head sensors

File: tobi_description/urdf/tobi_3of4.urdf.xacro (robot description, xacro)
@@ -133,5 +133,5 @@
     <parent link="box_head_link" />
     <child link="sensor_head_link" />
-    <origin xyz="0.08 0 0.20" rpy="0 0 0" />
+    <origin xyz="0.08 -0.5 0.20" rpy="0 0 0" />
   </joint>
 </robot>

Commit message: change box position

File: tobi_description/urdf/tobi_3of4.urdf.xacro (robot description, xacro)
@@ -133,5 +133,5 @@
     <parent link="box_head_link" />
     <child link="sensor_head_link" />
-    <origin xyz="0.08 -0.5 0.20" rpy="0 0 0" />
+    <origin xyz="0.08 0.1 0.20" rpy="0 0 0" />
   </joint>
 </robot>

Commit message: change parameter

File: tobi_description/urdf/tobi_3of4.urdf.xacro (robot description, xacro)
@@ -133,5 +133,5 @@
     <parent link="box_head_link" />
     <child link="sensor_head_link" />
-    <origin xyz="0.08 0.1 0.20" rpy="0 0 0" />
+    <origin xyz="0.08 0.02 0.20" rpy="0 0 0" />
   </joint>
 </robot>

Commit message: consistent guiabot 3of4

File: tobi_description/urdf/tobi_3of4.urdf.xacro (robot description, xacro)
@@ -60,7 +60,7 @@
     </visual>
     <visual>
-      <origin xyz="0.115 0.165 -0.01" rpy="0 -0.56 0" />
+      <origin xyz="0.125 0.165 -0.03" rpy="0 -0.56 0" />
       <geometry>
-        <cylinder radius="0.017" length="0.23"/>
+        <cylinder radius="0.017" length="0.25"/>
       </geometry>
       <material name="grey" >
@@ -69,7 +69,7 @@
     </visual>
     <visual>
-      <origin xyz="0.115 -0.165 -0.01" rpy="0 -0.56 0" />
+      <origin xyz="0.125 -0.165 -0.03" rpy="0 -0.56 0" />
       <geometry>
-        <cylinder radius="0.017" length="0.23"/>
+        <cylinder radius="0.017" length="0.25"/>
       </geometry>
       <material name="grey" >
@@ -92,13 +92,13 @@
     </collision>
     <collision>
-      <origin xyz="0.115 0.165 -0.01" rpy="0 -0.56 0" />
+      <origin xyz="0.125 0.165 -0.03" rpy="0 -0.56 0" />
       <geometry>
-        <cylinder radius="0.017" length="0.23"/>
+        <cylinder radius="0.017" length="0.25"/>
       </geometry>
     </collision>
     <collision>
-      <origin xyz="0.115 -0.165 -0.01" rpy="0 -0.56 0" />
+      <origin xyz="0.125 -0.165 -0.03" rpy="0 -0.56 0" />
       <geometry>
-        <cylinder radius="0.017" length="0.23"/>
+        <cylinder radius="0.017" length="0.25"/>
       </geometry>
     </collision>

Commit message: test arm position

File: tobi_description/urdf/tobi_3of4.urdf.xacro (robot description, xacro)
@@ -42,5 +42,5 @@
     <parent link="guiabot" />
     <child link="katana_base_link" />
-    <origin xyz="0.03 0 0.84" rpy="0 ${-M_PI/2} 0" />
+    <origin xyz="0.05 0 0.84" rpy="0 ${-M_PI/2} 0" />
   </joint>
   <link name="base_link" />

Commit message: change arm position

File: tobi_description/urdf/tobi_3of4.urdf.xacro (robot description, xacro)
@@ -42,5 +42,5 @@
     <parent link="guiabot" />
     <child link="katana_base_link" />
-    <origin xyz="0.05 0 0.84" rpy="0 ${-M_PI/2} 0" />
+    <origin xyz="0.02 0 0.84" rpy="0 ${-M_PI/2} 0" />
   </joint>
   <link name="base_link" />

Commit message: change arm position for 3of4

File: tobi_description/urdf/tobi_3of4.urdf.xacro (robot description, xacro)
@@ -42,5 +42,5 @@
     <parent link="guiabot" />
     <child link="katana_base_link" />
-    <origin xyz="0.02 0 0.84" rpy="0 ${-M_PI/2} 0" />
+    <origin xyz="0.01 0 0.84" rpy="0 ${-M_PI/2} 0" />
   </joint>
   <link name="base_link" />
