Commit message: fixed arm mounting position in urdf model.
Also fixed some arm poses.

File: tobi_description/urdf/tobi_2of4.urdf.xacro (robot description, xacro)
@@ -42,5 +42,5 @@
     <parent link="guiabot" />
     <child link="katana_base_link" />
-    <origin xyz=".02 0 0.84" rpy="0 ${-M_PI/2} 0" />
+    <origin xyz="-.02 0 0.84" rpy="0 ${-M_PI/2} 0" />
   </joint>
   <link name="base_link" />
@@ -113,5 +113,5 @@
     <parent link="katana_base_link" />
     <child link="box_head_link" />
-    <origin xyz="0.32 0 0.02" rpy="${M_PI} ${-M_PI/2} 0" />
+    <origin xyz="0.32 0 -0.02" rpy="${M_PI} ${-M_PI/2} 0" />
   </joint>
   <link name="sensor_head_link">

Commit message: refined robot collision models

File: tobi_description/urdf/tobi_2of4.urdf.xacro (robot description, xacro)
@@ -60,7 +60,7 @@
     </visual>
     <visual>
-      <origin xyz="0.11 0.165 0" rpy="0 -0.56 0" />
+      <origin xyz="0.115 0.165 -0.01" rpy="0 -0.56 0" />
       <geometry>
-        <cylinder radius="0.02" length="0.26"/>
+        <cylinder radius="0.017" length="0.23"/>
       </geometry>
       <material name="grey" >
@@ -69,7 +69,7 @@
     </visual>
     <visual>
-      <origin xyz="0.11 -0.165 0" rpy="0 -0.56 0" />
+      <origin xyz="0.115 -0.165 -0.01" rpy="0 -0.56 0" />
       <geometry>
-        <cylinder radius="0.02" length="0.26"/>
+        <cylinder radius="0.017" length="0.23"/>
       </geometry>
       <material name="grey" >
@@ -92,13 +92,13 @@
     </collision>
     <collision>
-      <origin xyz="0.11 0.165 0" rpy="0 -0.56 0" />
+      <origin xyz="0.115 0.165 -0.01" rpy="0 -0.56 0" />
       <geometry>
-        <cylinder radius="0.02" length="0.26"/>
+        <cylinder radius="0.017" length="0.23"/>
       </geometry>
     </collision>
     <collision>
-      <origin xyz="0.11 -0.165 0" rpy="0 -0.56 0" />
+      <origin xyz="0.115 -0.165 -0.01" rpy="0 -0.56 0" />
       <geometry>
-        <cylinder radius="0.02" length="0.26"/>
+        <cylinder radius="0.017" length="0.23"/>
       </geometry>
     </collision>

Commit message: refined collision model for tobi 2of4

File: tobi_description/urdf/tobi_2of4.urdf.xacro (robot description, xacro)
@@ -42,5 +42,5 @@
     <parent link="guiabot" />
     <child link="katana_base_link" />
-    <origin xyz="-.02 0 0.84" rpy="0 ${-M_PI/2} 0" />
+    <origin xyz="-0.01 0 0.86" rpy="0 ${-M_PI/2} 0" />
   </joint>
   <link name="base_link" />
@@ -60,7 +60,7 @@
     </visual>
     <visual>
-      <origin xyz="0.115 0.165 -0.01" rpy="0 -0.56 0" />
+      <origin xyz="0.125 0.165 -0.03" rpy="0 -0.56 0" />
       <geometry>
-        <cylinder radius="0.017" length="0.23"/>
+        <cylinder radius="0.017" length="0.25"/>
       </geometry>
       <material name="grey" >
@@ -69,7 +69,7 @@
     </visual>
     <visual>
-      <origin xyz="0.115 -0.165 -0.01" rpy="0 -0.56 0" />
+      <origin xyz="0.125 -0.165 -0.03" rpy="0 -0.56 0" />
       <geometry>
-        <cylinder radius="0.017" length="0.23"/>
+        <cylinder radius="0.017" length="0.25"/>
       </geometry>
       <material name="grey" >
@@ -92,13 +92,13 @@
     </collision>
     <collision>
-      <origin xyz="0.115 0.165 -0.01" rpy="0 -0.56 0" />
+      <origin xyz="0.125 0.165 -0.03" rpy="0 -0.56 0" />
       <geometry>
-        <cylinder radius="0.017" length="0.23"/>
+        <cylinder radius="0.017" length="0.25"/>
       </geometry>
     </collision>
     <collision>
-      <origin xyz="0.115 -0.165 -0.01" rpy="0 -0.56 0" />
+      <origin xyz="0.125 -0.165 -0.03" rpy="0 -0.56 0" />
       <geometry>
-        <cylinder radius="0.017" length="0.23"/>
+        <cylinder radius="0.017" length="0.25"/>
       </geometry>
     </collision>
@@ -113,5 +113,5 @@
     <parent link="katana_base_link" />
     <child link="box_head_link" />
-    <origin xyz="0.32 0 -0.02" rpy="${M_PI} ${-M_PI/2} 0" />
+    <origin xyz="0.3 0 -0.01" rpy="${M_PI} ${-M_PI/2} 0" />
   </joint>
   <link name="sensor_head_link">

Commit message: change stuff for second robot

File: tobi_description/urdf/tobi_2of4.urdf.xacro (robot description, xacro)
@@ -133,5 +133,5 @@
     <parent link="box_head_link" />
     <child link="sensor_head_link" />
-    <origin xyz="0.08 0 0.20" rpy="0 0 0" />
+    <origin xyz="0.08 0.02 0.20" rpy="0 0 0" />
   </joint>
 </robot>

Commit message: connect head directly to guiabot and not over the arm

File: tobi_description/urdf/tobi_2of4.urdf.xacro (robot description, xacro)
@@ -42,5 +42,5 @@
     <parent link="guiabot" />
     <child link="katana_base_link" />
-    <origin xyz="-0.01 0 0.86" rpy="0 ${-M_PI/2} 0" />
+    <origin xyz="0.0 0 0.86" rpy="0 ${-M_PI/2} 0" />
   </joint>
   <link name="base_link" />
@@ -111,7 +111,7 @@
   </link>
   <joint name="katana_link_to_box_head" type="fixed">
-    <parent link="katana_base_link" />
+    <parent link="guiabot" />
     <child link="box_head_link" />
-    <origin xyz="0.3 0 -0.01" rpy="${M_PI} ${-M_PI/2} 0" />
+    <origin xyz="0 0 1.16" rpy="0 0 ${M_PI}" />
   </joint>
   <link name="sensor_head_link">

File: tobi_description/urdf/tobi_3of4.urdf.xacro (robot description, xacro)
@@ -42,5 +42,5 @@
     <parent link="guiabot" />
     <child link="katana_base_link" />
-    <origin xyz="-.02 0 0.84" rpy="0 ${-M_PI/2} 0" />
+    <origin xyz="0.03 0 0.84" rpy="0 ${-M_PI/2} 0" />
   </joint>
   <link name="base_link" />
@@ -111,7 +111,7 @@
   </link>
   <joint name="katana_link_to_box_head" type="fixed">
-    <parent link="katana_base_link" />
+    <parent link="guiabot" />
     <child link="box_head_link" />
-    <origin xyz="0.32 0 -0.02" rpy="${M_PI} ${-M_PI/2} 0" />
+    <origin xyz="0 0 1.16" rpy="0 0 ${M_PI}" />
   </joint>
   <link name="sensor_head_link">

Commit message: changed box model due to collisions

File: tobi_description/urdf/tobi_2of4.urdf.xacro (robot description, xacro)
@@ -80,5 +80,5 @@
       <origin xyz="0.16 0 -0.15" rpy="0 0.08 0" />
       <geometry>
-        <box size="0.04 0.35 0.08"/>
+        <box size="0.04 0.31 0.08"/>
       </geometry>
       <material name="grey" >
@@ -106,5 +106,5 @@
       <origin xyz="0.16 0 -0.15" rpy="0 0.08 0" />
       <geometry>
-        <box size="0.04 0.35 0.08"/>
+        <box size="0.04 0.31 0.08"/>
       </geometry>
     </collision>

File: tobi_description/urdf/tobi_3of4.urdf.xacro (robot description, xacro)
@@ -80,5 +80,5 @@
       <origin xyz="0.16 0 -0.15" rpy="0 0.08 0" />
       <geometry>
-        <box size="0.04 0.35 0.08"/>
+        <box size="0.04 0.31 0.08"/>
       </geometry>
       <material name="grey" >
@@ -106,5 +106,5 @@
       <origin xyz="0.16 0 -0.15" rpy="0 0.08 0" />
       <geometry>
-        <box size="0.04 0.35 0.08"/>
+        <box size="0.04 0.31 0.08"/>
       </geometry>
     </collision>

Commit message: Revert "changed box model due to collisions"
This reverts commit 2543d1638f4517239f94cbcf0d9a41fc913b644b.

File: tobi_description/urdf/tobi_2of4.urdf.xacro (robot description, xacro)
@@ -80,5 +80,5 @@
       <origin xyz="0.16 0 -0.15" rpy="0 0.08 0" />
       <geometry>
-        <box size="0.04 0.31 0.08"/>
+        <box size="0.04 0.35 0.08"/>
       </geometry>
       <material name="grey" >
@@ -106,5 +106,5 @@
       <origin xyz="0.16 0 -0.15" rpy="0 0.08 0" />
       <geometry>
-        <box size="0.04 0.31 0.08"/>
+        <box size="0.04 0.35 0.08"/>
       </geometry>
     </collision>

File: tobi_description/urdf/tobi_3of4.urdf.xacro (robot description, xacro)
@@ -80,5 +80,5 @@
       <origin xyz="0.16 0 -0.15" rpy="0 0.08 0" />
       <geometry>
-        <box size="0.04 0.31 0.08"/>
+        <box size="0.04 0.35 0.08"/>
       </geometry>
       <material name="grey" >
@@ -106,5 +106,5 @@
       <origin xyz="0.16 0 -0.15" rpy="0 0.08 0" />
       <geometry>
-        <box size="0.04 0.31 0.08"/>
+        <box size="0.04 0.35 0.08"/>
       </geometry>
     </collision>

Commit message: adjusted the size of 'sensor_head_link' for both ToBi's

File: tobi_description/urdf/tobi_2of4.urdf.xacro (robot description, xacro)
@@ -118,5 +118,5 @@
     <visual>
       <geometry>
-        <box size="0.15 .30 .12"/>
+        <box size="0.15 .26 .12"/>
       </geometry>
       <material name="grey" >
@@ -126,5 +126,5 @@
     <collision>
       <geometry>
-        <box size="0.15 .30 .12"/>
+        <box size="0.15 .26 .12"/>
       </geometry>
     </collision>

File: tobi_description/urdf/tobi_3of4.urdf.xacro (robot description, xacro)
@@ -118,5 +118,5 @@
     <visual>
       <geometry>
-        <box size="0.15 .30 .12"/>
+        <box size="0.15 .26 .12"/>
       </geometry>
       <material name="grey" >
@@ -126,5 +126,5 @@
     <collision>
       <geometry>
-        <box size="0.15 .30 .12"/>
+        <box size="0.15 .26 .12"/>
       </geometry>
     </collision>

Commit message: moved katana_base_link in urdf -2cm along X-axis, changed xtion2 camera_mode from 1 to 5

File: tobi_description/urdf/tobi_2of4.urdf.xacro (robot description, xacro)
@@ -42,5 +42,5 @@
     <parent link="guiabot" />
     <child link="katana_base_link" />
-    <origin xyz="0.0 0 0.86" rpy="0 ${-M_PI/2} 0" />
+    <origin xyz="-0.02 0 0.86" rpy="0 ${-M_PI/2} 0" />
   </joint>
   <link name="base_link" />

Commit message: reverted hacks from competition: reset katana_base_link to 0 0 0.86

File: tobi_description/urdf/tobi_2of4.urdf.xacro (robot description, xacro)
@@ -42,5 +42,5 @@
     <parent link="guiabot" />
     <child link="katana_base_link" />
-    <origin xyz="-0.02 0 0.86" rpy="0 ${-M_PI/2} 0" />
+    <origin xyz="0 0 0.86" rpy="0 ${-M_PI/2} 0" />
   </joint>
   <link name="base_link" />

Commit message: katana_base_link mounted not exactly above base_link

File: tobi_description/urdf/tobi_2of4.urdf.xacro (robot description, xacro)
@@ -42,5 +42,5 @@
     <parent link="guiabot" />
     <child link="katana_base_link" />
-    <origin xyz="0 0 0.86" rpy="0 ${-M_PI/2} 0" />
+    <origin xyz="-0.02 0 0.86" rpy="0 ${-M_PI/2} 0" />
   </joint>
   <link name="base_link" />

Commit message: hopefully fixed urdf for katana_base_link

File: tobi_description/urdf/tobi_2of4.urdf.xacro (robot description, xacro)
@@ -42,5 +42,5 @@
     <parent link="guiabot" />
     <child link="katana_base_link" />
-    <origin xyz="-0.02 0 0.86" rpy="0 ${-M_PI/2} 0" />
+    <origin xyz="0.012 0 0.867" rpy="0 ${-M_PI/2} 0" />
   </joint>
   <link name="base_link" />
