Commit message: added tobi_2of4 with kinect for simulation

File: tobi_description/urdf/tobi_2of4_kinect.urdf.xacro (robot description, xacro)
@@ -1,8 +1,14 @@
 <?xml version="1.0"?>
 <robot
-  xmlns:xacro="http://ros.org/wiki/xacro"
+  xmlns:xacro="http://www.ros.org/wiki/xacro"
   xmlns:sensor="http://playerstage.sourceforge.net/gazebo/xmlschema/#sensor"
   xmlns:controller="http://playerstage.sourceforge.net/gazebo/xmlschema/#controller"
   name="tobi">
+  <!-- Import asus -->
+  <xacro:include filename="$(find tobi_description)/urdf/asus_camera.urdf.xacro" />
+  <!-- Import extra base -->
+  <!--xacro:include filename="$(find tobi_description)/urdf/tobi_2of4_kinect_base.urdf.xacro" /-->
+  <!-- Import gazebo setup -->
+  <xacro:include filename="$(find tobi_description)/urdf/gazebo.urdf.xacro"/>
   <xacro:macro name="box_inertial" params="x y z mass">
     <inertial>
@@ -116,12 +122,4 @@
   </joint>
   <link name="sensor_head_link">
-    <visual>
-      <geometry>
-        <box size="0.15 .26 .12"/>
-      </geometry>
-      <material name="grey" >
-        <color rgba="0.5 0.5 0.5 1" />
-      </material>
-    </visual>
     <collision>
       <geometry>
@@ -130,4 +128,7 @@
     </collision>
   </link>
+  <asus_camera name="xtion" parent="sensor_head_link">
+    <origin xyz="0 0 0" rpy="0 0.6 0"/>
+  </asus_camera>
   <joint name="box_head_to_sensor_head" type="fixed">
     <parent link="box_head_link" />

File: tobi_description/urdf/tobi_3of4.urdf.xacro (robot description, xacro)
@@ -14,5 +14,5 @@
     </inertial>
   </xacro:macro>
-  <property name="M_PI" value="3.1415926535897931" />
+  <xacro:property name="M_PI" value="3.1415926535897931" />
   <xacro:property name="guiabot_length" value="0.59"/>
   <xacro:property name="guiabot_width" value="0.48"/>
