Commit message: working, no gz

File: tobi_description/urdf/gazebo.urdf.xacro (robot description, xacro)
@@ -11,5 +11,5 @@
       <updateRate>30.0</updateRate>
     </plugin>
-   </gazebo>
+  </gazebo>
   <!-- gazebo>
 	    <plugin name="create_controller" filename="libgazebo_ros_create.so">
@@ -58,4 +58,4 @@
       <minDepth>0.001</minDepth>
       <maxVel>1.0</maxVel>
-    </gazebo-->
+    </gazebo>  /-->
 </robot>

File: tobi_description/urdf/tobi_2of4_kinect.urdf.xacro (robot description, xacro)
@@ -8,7 +8,9 @@
   <xacro:include filename="$(find tobi_description)/urdf/asus_camera.urdf.xacro" />
   <!-- Import extra base -->
-  <!--xacro:include filename="$(find tobi_description)/urdf/tobi_2of4_kinect_base.urdf.xacro" /-->
+  <xacro:include filename="$(find tobi_description)/urdf/tobi_2of4_kinect_base.urdf.xacro" />
   <!-- Import gazebo setup -->
-  <xacro:include filename="$(find tobi_description)/urdf/gazebo.urdf.xacro"/>
+  <!-- <xacro:include filename="$(find tobi_description)/urdf/gazebo.urdf.xacro"/>  -->
+  <!-- Import katana arm -->
+  <xacro:include filename="$(find katana_description)/urdf/katana_450_6m180_simple.urdf.xacro" />
   <xacro:macro name="box_inertial" params="x y z mass">
     <inertial>
@@ -44,6 +46,5 @@
   <!-- *** Neuronics Katana Arm *** -->
   <!-- **************************** -->
-  <xacro:include filename="$(find katana_description)/urdf/katana_450_6m180_simple.urdf.xacro" />
-  <joint name="tobi_guiabot_katana_joint" type="fixed">
+   <joint name="tobi_guiabot_katana_joint" type="fixed">
     <parent link="guiabot" />
     <child link="katana_base_link" />
@@ -51,5 +52,5 @@
   </joint>
   <link name="base_link" />
-  <joint name="base_link_to_guiabot" type="fixed">
+  <joint name="base_link_to_urdfguiabot" type="fixed">
     <parent link="base_link" />
     <child link="guiabot" />
@@ -80,5 +81,5 @@
       </geometry>
       <material name="grey" >
-        <color rgba="0.2 0.2 0.2 1" />
+        <color rgba="0.2 0.2 0.2 1"/>
       </material>
     </visual>
@@ -128,7 +129,4 @@
     </collision>
   </link>
-  <asus_camera name="xtion" parent="sensor_head_link">
-    <origin xyz="0 0 0" rpy="0 0.6 0"/>
-  </asus_camera>
   <joint name="box_head_to_sensor_head" type="fixed">
     <parent link="box_head_link" />
@@ -136,3 +134,6 @@
     <origin xyz="0.08 0.02 0.20" rpy="0 0 0" />
   </joint>
+   <xacro:asus_camera name="xtion" parent="sensor_head_link">
+    <origin xyz="0 0 0" rpy="0 0.6 0"/>
+  </xacro:asus_camera>
 </robot>

Commit message: fixed biron sim bot

File: tobi_description/urdf/gazebo.urdf.xacro (robot description, xacro)
@@ -1,8 +1,40 @@
 <?xml version="1.0"?>
-<robot xmlns:xacro="http://www.ros.org/wiki/xacro">
- <gazebo>
-   <!--plugin name="gazebo_ros_control" filename="libgazebo_ros_control.so">
-     <robotNamespace>/biron</robotNamespace>
-   </plugin-->
+<robot
+  xmlns:xacro="http://www.ros.org/wiki/xacro">
+  <gazebo>
+    <!-- <plugin name="gazebo_ros_control" filename="libgazebo_ros_control.so">
+      <robotNamespace>/biron</robotNamespace>
+    </plugin> -->
+    <plugin name="differential_drive_controller" filename="libgazebo_ros_diff_drive.so">
+      <legacyMode>false</legacyMode>
+      <alwaysOn>true</alwaysOn>
+      <updateRate>30</updateRate>
+      <leftJoint>left_wheel_joint</leftJoint>
+      <rightJoint>right_wheel_joint</rightJoint>
+      <wheelSeparation>0.4</wheelSeparation>
+      <wheelDiameter>0.086</wheelDiameter>
+      <torque>20</torque>
+      <commandTopic>cmd_vel</commandTopic>
+      <odometryTopic>odom</odometryTopic>
+      <odometryFrame>odom</odometryFrame>
+      <robotBaseFrame>base_link</robotBaseFrame>
+      <publishWheelTF>true</publishWheelTF>
+      <publishWheelJointState>false</publishWheelJointState>
+      <wheelAcceleration>1</wheelAcceleration>
+      <wheelTorque>5</wheelTorque>
+    </plugin>
+    <!-- <plugin name="create_controller" filename="libgazebo_ros_create.so">
+      <alwaysOn>true</alwaysOn>
+      <node_namespace>biron_node</node_namespace>
+      <left_wheel_joint>left_wheel_joint</left_wheel_joint>
+      <right_wheel_joint>right_wheel_joint</right_wheel_joint>
+      <front_castor_joint>front_castor_joint</front_castor_joint>
+      <rear_castor_joint>rear_castor_joint</rear_castor_joint>
+      <wheel_separation>.260</wheel_separation>
+      <wheel_diameter>0.066</wheel_diameter>
+      <base_geom>guiabot</base_geom>
+      <updateRate>40</updateRate>
+      <torque>1.0</torque>
+    </plugin> -->
     <plugin name="ground_truth" filename="libgazebo_ros_p3d.so">
       <frameName>map</frameName>
@@ -12,50 +44,97 @@
     </plugin>
   </gazebo>
-  <!-- gazebo>
-	    <plugin name="create_controller" filename="libgazebo_ros_create.so">
-	      <alwaysOn>true</alwaysOn>
-	      <node_namespace>biron_node</node_namespace>
-	      <left_wheel_joint>left_wheel_joint</left_wheel_joint>
-	      <right_wheel_joint>right_wheel_joint</right_wheel_joint>
-	      <front_castor_joint>front_castor_joint</front_castor_joint>
-	      <rear_castor_joint>rear_castor_joint</rear_castor_joint>
-	      <wheel_separation>.260</wheel_separation>
-	      <wheel_diameter>0.066</wheel_diameter>
-	      <base_geom>guiabot</base_geom>
-	      <updateRate>40</updateRate>
-	      <torque>1.0</torque>
-	    </plugin>
-	  </gazebo>
+   <gazebo reference="laser_front">
+    <sensor type="gpu_ray" name="sick_sensor">
+      <pose>0 0 0 0 0 0</pose>
+      <visualize>true</visualize>
+      <update_rate>30</update_rate>
+      <ray>
+        <scan>
+          <horizontal>
+            <samples>720</samples>
+            <resolution>1</resolution>
+            <min_angle>-1.570796</min_angle>
+            <max_angle>1.570796</max_angle>
+          </horizontal>
+        </scan>
+        <range>
+          <min>0.20</min>
+          <max>8.0</max>
+          <resolution>0.01</resolution>
+        </range>
+        <noise>
+          <type>gaussian</type>
+          <mean>0.0</mean>
+          <stddev>0.01</stddev>
+        </noise>
+      </ray>
+      <plugin name="laser_front_sick" filename="libgazebo_ros_gpu_laser.so">
+        <topicName>/scan</topicName>
+        <frameName>laser_front</frameName>
+      </plugin>
+    </sensor>
+  </gazebo>
+   <gazebo reference="laser_rear">
+    <sensor type="gpu_ray" name="hokuyo_sensor">
+      <pose>0 0 0 0 0 0</pose>
+      <visualize>false</visualize>
+      <update_rate>30</update_rate>
+      <ray>
+        <scan>
+          <horizontal>
+            <samples>720</samples>
+            <resolution>1</resolution>
+            <min_angle>-1.570796</min_angle>
+            <max_angle>1.570796</max_angle>
+          </horizontal>
+        </scan>
+        <range>
+          <min>0.20</min>
+          <max>4.0</max>
+          <resolution>0.01</resolution>
+        </range>
+        <noise>
+          <type>gaussian</type>
+          <mean>0.0</mean>
+          <stddev>0.01</stddev>
+        </noise>
+      </ray>
+      <plugin name="laser_rear_hokuyo" filename="libgazebo_ros_gpu_laser.so">
+        <topicName>/scan_rear</topicName>
+        <frameName>laser_rear</frameName>
+      </plugin>
+    </sensor>
+  </gazebo>
   <gazebo reference="left_wheel_link">
-      <mu1>1.0</mu1>
-      <mu2>1.0</mu2>
-      <kp>1000000.0</kp>
-      <kd>100.0</kd>
-      <minDepth>0.001</minDepth>
-      <maxVel>1.0</maxVel>
-    </gazebo>
-    <gazebo reference="right_wheel_link">
-      <mu1>1.0</mu1>
-      <mu2>1.0</mu2>
-      <kp>1000000.0</kp>
-      <kd>100.0</kd>
-      <minDepth>0.001</minDepth>
-      <maxVel>1.0</maxVel>
-    </gazebo>
-    <gazebo reference="rear_wheel_link">
-      <mu1>0.0</mu1>
-      <mu2>0.0</mu2>
-      <kp>1000000.0</kp>
-      <kd>100.0</kd>
-      <minDepth>0.001</minDepth>
-      <maxVel>1.0</maxVel>
-    </gazebo>
-    <gazebo reference="front_wheel_link">
-      <mu1>0.0</mu1>
-      <mu2>0.0</mu2>
-      <kp>1000000.0</kp>
-      <kd>100.0</kd>
-      <minDepth>0.001</minDepth>
-      <maxVel>1.0</maxVel>
-    </gazebo>  /-->
+    <mu1>1.0</mu1>
+    <mu2>1.0</mu2>
+    <kp>1000000.0</kp>
+    <kd>100.0</kd>
+    <minDepth>0.001</minDepth>
+    <maxVel>1.0</maxVel>
+  </gazebo>
+  <gazebo reference="right_wheel_link">
+    <mu1>1.0</mu1>
+    <mu2>1.0</mu2>
+    <kp>1000000.0</kp>
+    <kd>100.0</kd>
+    <minDepth>0.001</minDepth>
+    <maxVel>1.0</maxVel>
+  </gazebo>
+  <gazebo reference="rear_wheel_link">
+    <mu1>0.0</mu1>
+    <mu2>0.0</mu2>
+    <kp>1000000.0</kp>
+    <kd>100.0</kd>
+    <minDepth>0.001</minDepth>
+    <maxVel>1.0</maxVel>
+  </gazebo>
+  <gazebo reference="front_wheel_link">
+    <mu1>0.0</mu1>
+    <mu2>0.0</mu2>
+    <kp>1000000.0</kp>
+    <kd>100.0</kd>
+    <minDepth>0.001</minDepth>
+    <maxVel>1.0</maxVel>
+  </gazebo>
 </robot>

File: tobi_description/urdf/tobi_2of4_kinect.urdf.xacro (robot description, xacro)
@@ -8,9 +8,9 @@
   <xacro:include filename="$(find tobi_description)/urdf/asus_camera.urdf.xacro" />
   <!-- Import extra base -->
-  <xacro:include filename="$(find tobi_description)/urdf/tobi_2of4_kinect_base.urdf.xacro" />
+   <xacro:include filename="$(find tobi_description)/urdf/tobi_2of4_kinect_base.urdf.xacro" />
   <!-- Import gazebo setup -->
-  <!-- <xacro:include filename="$(find tobi_description)/urdf/gazebo.urdf.xacro"/>  -->
+    <xacro:include filename="$(find tobi_description)/urdf/gazebo.urdf.xacro"/>
   <!-- Import katana arm -->
-  <xacro:include filename="$(find katana_description)/urdf/katana_450_6m180_simple.urdf.xacro" />
+    <xacro:include filename="$(find katana_description)/urdf/katana_450_6m180_simple.urdf.xacro" />
   <xacro:macro name="box_inertial" params="x y z mass">
     <inertial>
@@ -46,5 +46,5 @@
   <!-- *** Neuronics Katana Arm *** -->
   <!-- **************************** -->
-   <joint name="tobi_guiabot_katana_joint" type="fixed">
+     <joint name="tobi_guiabot_katana_joint" type="fixed">
     <parent link="guiabot" />
     <child link="katana_base_link" />

File: tobi_description/urdf/tobi_2of4_kinect_base.urdf.xacro (robot description, xacro)
@@ -1,4 +1,9 @@
 <?xml version="1.0" ?>
-<robot>
+<robot xmlns:xacro="http://www.ros.org/wiki/xacro">
+<xacro:property name="caster_radius" value="0.010"/>
+<xacro:property name="caster_seperation" value="0.40"/>
+<xacro:property name="wheel_seperation" value="0.40"/>
+<xacro:property name="wheel_radius" value="0.042"/>
+<xacro:property name="wheel_add_z" value="-0.005"/>
 <link name="left_wheel_link">
 	    <inertial>
@@ -11,5 +16,5 @@
 	      <origin xyz="0 0 0" rpy="0 1.5707 1.5707" />
 	      <geometry>
-	        <cylinder radius="0.033" length = "0.023"/>
+	        <cylinder radius="${wheel_radius}" length="0.023"/>
 	      </geometry>
 	    </visual>
@@ -17,10 +22,10 @@
 	      <origin xyz="0 0 0" rpy="0 1.5707 1.5707" />
 	      <geometry>
-	        <cylinder radius="0.033" length = "0.023"/>
+	        <cylinder radius="${wheel_radius}" length="0.023"/>
 	      </geometry>
 	    </collision>
 	  </link>
 	  <joint name="left_wheel_joint" type="continuous">
-	    <origin xyz="0 0.13 0.015" rpy="0 0 0"/>
+	    <origin xyz="0 ${wheel_seperation/2} ${wheel_radius+wheel_add_z}" rpy="0 0 0"/>
 	    <parent link="base_link"/>
 	    <child link="left_wheel_link"/>
@@ -37,5 +42,5 @@
 	      <origin xyz="0 0 0" rpy="0 1.5707 1.5707" />
 	      <geometry>
-	        <cylinder radius="0.033" length = "0.023"/>
+	        <cylinder radius="${wheel_radius}" length="0.023"/>
 	      </geometry>
 	    </visual>
@@ -43,14 +48,15 @@
 	      <origin xyz="0 0 0" rpy="0 1.5707 1.5707" />
 	      <geometry>
-	        <cylinder radius="0.033" length = "0.023"/>
+	        <cylinder radius="${wheel_radius}" length="0.023"/>
 	      </geometry>
 	    </collision>
 	  </link>
 	  <joint name="right_wheel_joint" type="continuous">
-	    <origin xyz="0 -0.13 0.015" rpy="0 0 0"/>
+	    <origin xyz="0 ${-wheel_seperation/2} ${wheel_radius+wheel_add_z}" rpy="0 0 0"/>
 	    <parent link="base_link"/>
 	    <child link="right_wheel_link"/>
 	    <axis xyz="0 1 0"/>
 	  </joint>
+	<!-- CASTORS -->
 	  <link name="rear_wheel_link">
 	    <inertial>
@@ -63,5 +69,5 @@
 	      <origin xyz="0 0 0" rpy="0 1.5707 1.5707"/>
 	      <geometry>
-	        <sphere radius="0.015" />
+	        <sphere radius="${caster_radius}" />
 	      </geometry>
 	    </visual>
@@ -69,5 +75,5 @@
 	      <origin xyz="0 0 0" rpy="0 1.5707 1.5707" />
 	      <geometry>
-	        <sphere radius="0.015" />
+	        <sphere radius="${caster_radius}" />
 	      </geometry>
 	    </collision>
@@ -75,5 +81,5 @@
 	  <!-- fixed because there's no transmission -->
 	  <joint name="rear_castor_joint" type="fixed">
-	    <origin xyz="-0.13 0 0.0" rpy="0 0 0"/>
+	    <origin xyz="${-caster_seperation/2} 0 ${caster_radius+wheel_add_z}" rpy="0 0 0"/>
 	    <parent link="base_link"/>
 	    <child link="rear_wheel_link"/>
@@ -90,5 +96,5 @@
 	      <origin xyz="0 0 0" rpy="0 1.5707 1.5707"/>
 	      <geometry>
-	        <sphere radius="0.018" />
+	        <sphere radius="${caster_radius}" />
 	      </geometry>
 	    </visual>
@@ -96,5 +102,5 @@
 	      <origin xyz="0 0 0" rpy="0 1.5707 1.5707" />
 	      <geometry>
-	        <sphere radius="0.018" />
+	        <sphere radius="${caster_radius}" />
 	      </geometry>
 	    </collision>
@@ -102,8 +108,61 @@
 	  <!-- fixed because there's no transmission -->
 	  <joint name="front_castor_joint" type="fixed">
-	    <origin xyz="0.13 0 0.0" rpy="0 0 0"/>
+	    <origin xyz="${caster_seperation/2} 0 ${caster_radius+wheel_add_z}" rpy="0 0 0"/>
 	    <parent link="base_link"/>
 	    <child link="front_wheel_link"/>
 	    <axis xyz="0 1 0"/>
 	  </joint>
+<!-- Laser links-->
+		<joint name="sick_joint" type="fixed">
+    <axis xyz="0 0 0" />
+    <origin xyz="0.05 0 0.30" rpy="0 0 0"/>
+    <parent link="base_link"/>
+    <child link="laser_front"/>
+  </joint>
+	<joint name="hokuyo_joint" type="fixed">
+    <axis xyz="0 0 0" />
+    <origin xyz="-0.05 0 0.30" rpy="0 0 ${M_PI}"/>
+    <parent link="base_link"/>
+    <child link="laser_rear"/>
+  </joint>
+		<!-- Hokuyo Laser -->
+  <link name="laser_rear">
+    <collision>
+      <origin xyz="0 0 0" rpy="0 0 0"/>
+      <geometry>
+    <box size="0.01 0.01 0.01"/>
+      </geometry>
+    </collision>
+    <visual>
+      <origin xyz="0 0 0" rpy="0 0 0"/>
+      <geometry>
+        <box size="0.01 0.01 0.01"/>
+      </geometry>
+    </visual>
+    <inertial>
+      <mass value="1e-5" />
+      <origin xyz="0 0 0" rpy="0 0 0"/>
+      <inertia ixx="1e-6" ixy="0" ixz="0" iyy="1e-6" iyz="0" izz="1e-6" />
+    </inertial>
+  </link>
+	<!-- Hokuyo Laser -->
+  <link name="laser_front">
+    <collision>
+      <origin xyz="0 0 0" rpy="0 0 0"/>
+      <geometry>
+    <box size="0.01 0.01 0.01"/>
+      </geometry>
+    </collision>
+    <visual>
+      <origin xyz="0 0 0" rpy="0 0 0"/>
+      <geometry>
+        <box size="0.01 0.01 0.01"/>
+      </geometry>
+    </visual>
+    <inertial>
+      <mass value="1e-5" />
+      <origin xyz="0 0 0" rpy="0 0 0"/>
+      <inertia ixx="1e-6" ixy="0" ixz="0" iyy="1e-6" iyz="0" izz="1e-6" />
+    </inertial>
+  </link>
 </robot>
