Commit message: fixed wrong path

File: tobi_description/urdf/asus_camera.urdf.xacro (robot description, xacro)
@@ -17,5 +17,5 @@
           <origin xyz="0 0 0" rpy="0 0 0" />
           <geometry>
-            <mesh filename="package://tobi_world_misc/meshes/asus_camera/asus_camera_simple.dae"/>
+            <mesh filename="package://tobi_description/meshes/asus_camera/asus_camera_simple.dae"/>
           </geometry>
         </visual>

File: tobi_description/urdf/gazebo.urdf.xacro (robot description, xacro)
@@ -16,5 +16,5 @@
       <torque>20</torque>
       <commandTopic>cmd_vel</commandTopic>
-      <odometryTopic>odom</odometryTopic>
+      <odometryTopic>map</odometryTopic>
       <odometryFrame>odom</odometryFrame>
       <robotBaseFrame>base_link</robotBaseFrame>
